File: PCBs/DNMS - T4+NodeMCU/DNMS - T4+NodeMCU V1.2/DNMS.sch (KiCad schematic (older format))
At the start: 12 parts, among them J1 Conn_2Rows-07Pins, J2 Conn_01x02, J3 Conn_01x04, J4 Conn_01x05, U1 NodeMCU V2, U2 NodeMCU V3, U3 Teensy4.0

Commit message: change connector to mic to molex pico-ezmate
move other connectors around
Parts:
- removed J1: Conn_2Rows-07Pins, Connector_PinHeader_2.54mm:PinHeader_2x03_P2.54mm_Vertical, symbol Connector_Generic:Conn_2Rows-07Pins
- removed U1: NodeMCU V2, nodemcu:NodeMCU_Amica_R2, symbol nodemcu:NodeMCU_Amica_R2
- added C4, C5, C7: 100nF, Capacitor_SMD:C_0603_1608Metric_Pad1.05x0.95mm_HandSolder, symbol Device:C
- added C6: 10uF, Capacitor_SMD:C_0805_2012Metric_Pad1.15x1.40mm_HandSolder, symbol Device:C
- added J1: Conn_02x03_Odd_Even, Connector_PinHeader_2.54mm:PinHeader_2x03_P2.54mm_Vertical, symbol Connector_Generic:Conn_02x03_Odd_Even
- C1, C2, C3: footprint Capacitor_THT:C_Rect_L7.0mm_W2.0mm_P5.00mm -> Capacitor_SMD:C_0603_1608Metric_Pad1.05x0.95mm_HandSolder
- R1, R2: footprint Resistor_THT:R_Axial_DIN0207_L6.3mm_D2.5mm_P10.16mm_Horizontal -> Resistor_SMD:R_0603_1608Metric_Pad1.05x0.95mm_HandSolder
Connections:
- wire segments 100 -> 47
- no-connect marks 62 -> 59
