File: PCBs/DNMS - T4+NodeMCUv3/DNMS - T4+NodeMCUv3 v1.0/DNMS.kicad_pcb (KiCad board)
At the start: 2 copper layers, 60 x 32.5 mm, 23 parts, among them J1 Conn_01x06, J2 Conn_01x02, J3 Conn_01x04, J4 Conn_01x05, J5 Conn_01x06, J6 Conn_01x05, U2 NodeMCU V3, U3 Teensy4.0

Commit message: move component
Parts:
- moved C3 3.57 mm to (110.4, 83.8), turned to 180 degrees
Routing:
- net +5V: track 105.6 -> 107.8 mm
